Commit message: fix pi

File: src/crab_description/models/crab_model.xacro (robot description, xacro)
@@ -19,6 +19,5 @@
     		</visual>
 	</link>
-<!-- Pi parameter -->
-	<xacro:property name="pi" value="3.1415926535897931" />
+<!-- Pi is already defined globally in xacro, using it directly -->
 <!-- Joint properties -->
 	<xacro:property name="joint_lower_limit" value="-${1.5}" />

Commit message: new parametrs

File: src/crab_description/models/crab_model.xacro (robot description, xacro)
@@ -1,4 +1,18 @@
 <?xml version="1.0"?>
 <robot xmlns:xacro="http://ros.org/wiki/xacro" name="crab">
+<!-- ============================================================================ -->
+<!-- РАЗМЕРЫ ЗВЕНЬЕВ НОГИ (в метрах) -->
+<!-- ============================================================================ -->
+	<xacro:property name="coxa_length" value="0.025" />   <!-- 25 мм: ось coxa → ось femur -->
+	<xacro:property name="femur_length" value="0.077" />  <!-- 77 мм: ось femur → ось tibia -->
+	<xacro:property name="tibia_length" value="0.120" />  <!-- 120 мм: ось tibia → кончик -->
+	<!-- Суммарная длина ноги: 0.025 + 0.077 + 0.120 = 0.222 м -->
+<!-- ============================================================================ -->
+<!-- ГЕОМЕТРИЯ ТЕЛА -->
+<!-- ============================================================================ -->
+	<!-- Позиции крепления ног (leg_center) относительно центра тела -->
+	<xacro:property name="body_front_x" value="0.087598" />
+	<xacro:property name="body_side_y" value="0.050575" />
+	<xacro:property name="body_mid_y" value="0.06985" />
 <!-- Build the body frame -->
 	<link name="base_link" />
@@ -19,5 +33,4 @@
     		</visual>
 	</link>
-<!-- Pi is already defined globally in xacro, using it directly -->
 <!-- Joint properties -->
 	<xacro:property name="joint_lower_limit" value="-${1.5}" />
@@ -53,5 +66,5 @@
   	</link>
   	<joint name="femur_joint_${side}${num}" type="revolute">
-    		<origin xyz="0.0294 0 0" rpy="-${pi/2} 0 0" />
+    		<origin xyz="${coxa_length} 0 0" rpy="-${pi/2} 0 0" />
     		<parent link="coxa_${side}${num}" />
     		<child link="femur_${side}${num}" />
@@ -71,5 +84,5 @@
   	</link>
   	<joint name="tibia_joint_${side}${num}" type="revolute">
-    		<origin xyz="0.08 0 0" rpy="${pi} 0 ${pi/2}" />
+    		<origin xyz="${femur_length} 0 0" rpy="${pi} 0 ${pi/2}" />
     		<parent link="femur_${side}${num}" />
     		<child link="tibia_${side}${num}" />
@@ -89,5 +102,5 @@
   	</link>
   	<joint name="tibia_foot_joint_${side}${num}" type="fixed">
-    		<origin xyz="0.117 0 0" rpy="0 0 0" />
+    		<origin xyz="${tibia_length} 0 0" rpy="0 0 0" />
     		<parent link="tibia_${side}${num}" />
     		<child link="tibia_foot_${side}${num}" />

Commit message: fix

File: src/crab_description/models/crab_model.xacro (robot description, xacro)
@@ -1,10 +1,12 @@
 <?xml version="1.0"?>
 <robot xmlns:xacro="http://ros.org/wiki/xacro" name="crab">
+	<xacro:arg name="config" default="$(find crab_description)/config/robot_geometry.yaml" />
+	<xacro:property name="cfg" value="${xacro.load_yaml(config)}" />
 <!-- ============================================================================ -->
 <!-- РАЗМЕРЫ ЗВЕНЬЕВ НОГИ (в метрах) -->
 <!-- ============================================================================ -->
-	<xacro:property name="coxa_length" value="0.025" />   <!-- 25 мм: ось coxa → ось femur -->
-	<xacro:property name="femur_length" value="0.077" />  <!-- 77 мм: ось femur → ось tibia -->
-	<xacro:property name="tibia_length" value="0.120" />  <!-- 120 мм: ось tibia → кончик -->
+	<xacro:property name="coxa_length" value="${cfg['leg']['coxa_length']}" />   <!-- 25 мм: ось coxa → ось femur -->
+	<xacro:property name="femur_length" value="${cfg['leg']['femur_length']}" />  <!-- 77 мм: ось femur → ось tibia -->
+	<xacro:property name="tibia_length" value="${cfg['leg']['tibia_length']}" />  <!-- 120 мм: ось tibia → кончик -->
 	<!-- Суммарная длина ноги: 0.025 + 0.077 + 0.120 = 0.222 м -->
 <!-- ============================================================================ -->
@@ -34,6 +36,6 @@
 	</link>
 <!-- Joint properties -->
-	<xacro:property name="joint_lower_limit" value="-${1.5}" />
-	<xacro:property name="joint_upper_limit" value="${1.5}" />
+	<xacro:property name="joint_lower_limit" value="${cfg['joint_limits']['lower']}" />
+	<xacro:property name="joint_upper_limit" value="${cfg['joint_limits']['upper']}" />
 	<xacro:property name="joint_effort" value="10000" />
 	<xacro:property name="joint_velocity" value="100" />

Commit message: fix rviz

File: src/crab_description/models/crab_model.xacro (robot description, xacro)
@@ -1,12 +1,15 @@
 <?xml version="1.0"?>
 <robot xmlns:xacro="http://ros.org/wiki/xacro" name="crab">
-	<xacro:arg name="config" default="$(find-pkg-share crab_description)/config/robot_geometry.yaml" />
-	<xacro:property name="cfg" value="${xacro.load_yaml(config)}" />
+	<xacro:arg name="coxa_length" default="0.025" />
+	<xacro:arg name="femur_length" default="0.077" />
+	<xacro:arg name="tibia_length" default="0.120" />
+	<xacro:arg name="joint_lower_limit" default="-1.5" />
+	<xacro:arg name="joint_upper_limit" default="1.5" />
 <!-- ============================================================================ -->
 <!-- РАЗМЕРЫ ЗВЕНЬЕВ НОГИ (в метрах) -->
 <!-- ============================================================================ -->
-	<xacro:property name="coxa_length" value="${cfg['leg']['coxa_length']}" />   <!-- 25 мм: ось coxa → ось femur -->
-	<xacro:property name="femur_length" value="${cfg['leg']['femur_length']}" />  <!-- 77 мм: ось femur → ось tibia -->
-	<xacro:property name="tibia_length" value="${cfg['leg']['tibia_length']}" />  <!-- 120 мм: ось tibia → кончик -->
+	<xacro:property name="coxa_length" value="${coxa_length}" />   <!-- 25 мм: ось coxa → ось femur -->
+	<xacro:property name="femur_length" value="${femur_length}" />  <!-- 77 мм: ось femur → ось tibia -->
+	<xacro:property name="tibia_length" value="${tibia_length}" />  <!-- 120 мм: ось tibia → кончик -->
 	<!-- Суммарная длина ноги: 0.025 + 0.077 + 0.120 = 0.222 м -->
 <!-- ============================================================================ -->
@@ -36,6 +39,6 @@
 	</link>
 <!-- Joint properties -->
-	<xacro:property name="joint_lower_limit" value="${cfg['joint_limits']['lower']}" />
-	<xacro:property name="joint_upper_limit" value="${cfg['joint_limits']['upper']}" />
+	<xacro:property name="joint_lower_limit" value="${joint_lower_limit}" />
+	<xacro:property name="joint_upper_limit" value="${joint_upper_limit}" />
 	<xacro:property name="joint_effort" value="10000" />
 	<xacro:property name="joint_velocity" value="100" />

Commit message: add primitives

File: src/crab_description/models/crab_model.xacro (robot description, xacro)
@@ -6,4 +6,5 @@
 	<xacro:arg name="joint_lower_limit" default="-1.5" />
 	<xacro:arg name="joint_upper_limit" default="1.5" />
+	<xacro:arg name="use_primitives" default="false" />
 <!-- ============================================================================ -->
 <!-- РАЗМЕРЫ ЗВЕНЬЕВ НОГИ (в метрах) -->
@@ -31,5 +32,10 @@
       			<origin	xyz="0 0 0" rpy="0 0 0" />
       			<geometry>
-				<mesh filename="package://crab_description/meshes/thorax.STL" />
+				<xacro:if value="${use_primitives}">
+					<box size="0.18 0.12 0.04" />
+				</xacro:if>
+				<xacro:unless value="${use_primitives}">
+					<mesh filename="package://crab_description/meshes/thorax.STL" />
+				</xacro:unless>
       			</geometry>
      			<material name="grey">
@@ -63,5 +69,10 @@
       			<origin xyz="0 0 0" rpy="0 0 0" />
       			<geometry>
-        			<mesh filename="package://crab_description/meshes/coxa_${side}.STL" />
+					<xacro:if value="${use_primitives}">
+						<box size="${coxa_length} 0.02 0.02" />
+					</xacro:if>
+					<xacro:unless value="${use_primitives}">
+        				<mesh filename="package://crab_description/meshes/coxa_${side}.STL" />
+					</xacro:unless>
       			</geometry>
       			<material name="">
@@ -81,5 +92,10 @@
       			<origin xyz="0 0 0" rpy="0 0 0" />
       			<geometry>
-        			<mesh filename="package://crab_description/meshes/femur_${side}.STL" />
+					<xacro:if value="${use_primitives}">
+						<box size="${femur_length} 0.02 0.02" />
+					</xacro:if>
+					<xacro:unless value="${use_primitives}">
+        				<mesh filename="package://crab_description/meshes/femur_${side}.STL" />
+					</xacro:unless>
       			</geometry>
       			<material name="">
@@ -99,5 +115,10 @@
       			<origin xyz="0 0 0" rpy="0 0 0.06" />
       			<geometry>
-       				<mesh filename="package://crab_description/meshes/tibia_${side}.STL" />
+					<xacro:if value="${use_primitives}">
+						<box size="${tibia_length} 0.02 0.02" />
+					</xacro:if>
+					<xacro:unless value="${use_primitives}">
+       					<mesh filename="package://crab_description/meshes/tibia_${side}.STL" />
+					</xacro:unless>
       			</geometry>
       			<material name="">

Commit message: fix

File: src/crab_description/models/crab_model.xacro (robot description, xacro)
@@ -45,6 +45,6 @@
 	</link>
 <!-- Joint properties -->
-	<xacro:property name="joint_lower_limit" value="${joint_lower_limit}" />
-	<xacro:property name="joint_upper_limit" value="${joint_upper_limit}" />
+	<xacro:property name="joint_lower_limit_val" value="${xacro.arg('joint_lower_limit')}" />
+	<xacro:property name="joint_upper_limit_val" value="${xacro.arg('joint_upper_limit')}" />
 	<xacro:property name="joint_effort" value="10000" />
 	<xacro:property name="joint_velocity" value="100" />
@@ -63,5 +63,5 @@
     		<child link="coxa_${side}${num}" />
     		<axis xyz="0 0 -1" />
-    		<limit lower="${joint_lower_limit}" upper="${joint_upper_limit}" effort="${joint_effort}" velocity="${joint_velocity}" />
+    		<limit lower="${joint_lower_limit_val}" upper="${joint_upper_limit_val}" effort="${joint_effort}" velocity="${joint_velocity}" />
   	</joint>
   	<link name="coxa_${side}${num}">
@@ -86,5 +86,5 @@
     		<child link="femur_${side}${num}" />
     		<axis xyz="0 0 -1" />
-    		<limit lower="${joint_lower_limit}" upper="${joint_upper_limit}" effort="${joint_effort}" velocity="${joint_velocity}" />
+    		<limit lower="${joint_lower_limit_val}" upper="${joint_upper_limit_val}" effort="${joint_effort}" velocity="${joint_velocity}" />
   	</joint>
   	<link name="femur_${side}${num}">
@@ -109,5 +109,5 @@
     		<child link="tibia_${side}${num}" />
     		<axis xyz="0 0 1" />
-    		<limit lower="${joint_lower_limit}" upper="${joint_upper_limit}" effort="${joint_effort}" velocity="${joint_velocity}" />
+    		<limit lower="${joint_lower_limit_val}" upper="${joint_upper_limit_val}" effort="${joint_effort}" velocity="${joint_velocity}" />
   	</joint>
   	<link name="tibia_${side}${num}">

Commit message: fix

File: src/crab_description/models/crab_model.xacro (robot description, xacro)
@@ -10,7 +10,7 @@
 <!-- РАЗМЕРЫ ЗВЕНЬЕВ НОГИ (в метрах) -->
 <!-- ============================================================================ -->
-	<xacro:property name="coxa_length" value="${coxa_length}" />   <!-- 25 мм: ось coxa → ось femur -->
-	<xacro:property name="femur_length" value="${femur_length}" />  <!-- 77 мм: ось femur → ось tibia -->
-	<xacro:property name="tibia_length" value="${tibia_length}" />  <!-- 120 мм: ось tibia → кончик -->
+	<xacro:property name="coxa_length_val" value="${xacro.arg('coxa_length')}" />   <!-- 25 мм: ось coxa → ось femur -->
+	<xacro:property name="femur_length_val" value="${xacro.arg('femur_length')}" />  <!-- 77 мм: ось femur → ось tibia -->
+	<xacro:property name="tibia_length_val" value="${xacro.arg('tibia_length')}" />  <!-- 120 мм: ось tibia → кончик -->
 	<!-- Суммарная длина ноги: 0.025 + 0.077 + 0.120 = 0.222 м -->
 <!-- ============================================================================ -->
@@ -70,5 +70,5 @@
       			<geometry>
 					<xacro:if value="${xacro.arg('use_primitives') == 'true'}">
-						<box size="${coxa_length} 0.02 0.02" />
+						<box size="${coxa_length_val} 0.02 0.02" />
 					</xacro:if>
 					<xacro:unless value="${xacro.arg('use_primitives') == 'true'}">
@@ -82,5 +82,5 @@
   	</link>
   	<joint name="femur_joint_${side}${num}" type="revolute">
-    		<origin xyz="${coxa_length} 0 0" rpy="-${pi/2} 0 0" />
+    		<origin xyz="${coxa_length_val} 0 0" rpy="-${pi/2} 0 0" />
     		<parent link="coxa_${side}${num}" />
     		<child link="femur_${side}${num}" />
@@ -93,5 +93,5 @@
       			<geometry>
 					<xacro:if value="${xacro.arg('use_primitives') == 'true'}">
-						<box size="${femur_length} 0.02 0.02" />
+						<box size="${femur_length_val} 0.02 0.02" />
 					</xacro:if>
 					<xacro:unless value="${xacro.arg('use_primitives') == 'true'}">
@@ -105,5 +105,5 @@
   	</link>
   	<joint name="tibia_joint_${side}${num}" type="revolute">
-    		<origin xyz="${femur_length} 0 0" rpy="${pi} 0 ${pi/2}" />
+    		<origin xyz="${femur_length_val} 0 0" rpy="${pi} 0 ${pi/2}" />
     		<parent link="femur_${side}${num}" />
     		<child link="tibia_${side}${num}" />
@@ -116,5 +116,5 @@
       			<geometry>
 					<xacro:if value="${xacro.arg('use_primitives') == 'true'}">
-						<box size="${tibia_length} 0.02 0.02" />
+						<box size="${tibia_length_val} 0.02 0.02" />
 					</xacro:if>
 					<xacro:unless value="${xacro.arg('use_primitives') == 'true'}">
@@ -128,5 +128,5 @@
   	</link>
   	<joint name="tibia_foot_joint_${side}${num}" type="fixed">
-    		<origin xyz="${tibia_length} 0 0" rpy="0 0 0" />
+    		<origin xyz="${tibia_length_val} 0 0" rpy="0 0 0" />
     		<parent link="tibia_${side}${num}" />
     		<child link="tibia_foot_${side}${num}" />
